File: pcb/carry/Carry/Carry.kicad_sch (KiCad schematic)
At the start: 10 parts, among them J1 Conn_01x20_MountingPin, J2 Conn_01x02, U1 Luckfox-Pico_Mini_B, U2 MCP73831-2-OT

Commit message: updated
Parts:
- removed C1: C, symbol Device:C
- removed J1: Conn_01x20_MountingPin, symbol Connector_Generic_MountingPin:Conn_01x20_MountingPin
- removed TP1: TestPoint, symbol Connector:TestPoint
- U1: footprint (none) -> My_Custom_Parts:Luckfox_Pico_Mini_B
Connections:
- net GND: now also U2.2 (V_{SS}); no longer U1.2 (GND)
- net at J2.1 (Pin_1), U1.1 (VBUS), U2.3 (V_{BAT}): now also U2.4 (V_{DD})
- no-connect marks 0 -> 17

Commit message: updated
Connections:
- net GND: now also U1.2 (GND), U1.21 (GND)
- no-connect marks 17 -> 15
Changed lines of the file:
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@@
-	)
-	(no_connect
-		(at 140.97 63.5)
 	)
 	(no_connect
@@
 	(no_connect
 		(at 171.45 86.36)
-	)
-	(no_connect
-		(at 171.45 63.5)
 	)
 	(no_connect
@@
 	(symbol
 		(lib_id "power:GND")
+		(at 171.45 63.5 90)
+		(unit 1)
+		(body_style 1)
+		(exclude_from_sim no)
+		(in_bom yes)
+		(on_board yes)
+		(in_pos_files yes)
+		(dnp no)
+		(fields_autoplaced yes)
+		(property "Reference" "#PWR07"
+			(at 177.8 63.5 0)
+			(hide yes)
+			(show_name no)
+			(do_not_autoplace no)
+			(effects
+				(font
+					(size 1.27 1.27)
+				)
+			)
+		)
+		(property "Value" "GND"
+			(at 175.26 63.4999 90)
+			(show_name no)
+			(do_not_autoplace no)
+			(effects
+				(font
+					(size 1.27 1.27)
+				)
+				(justify right)
+			)
+		)
+		(property "Footprint" ""
+			(at 171.45 63.5 0)
+			(hide yes)
+			(show_name no)
+			(do_not_autoplace no)
+			(effects
+				(font
+					(size 1.27 1.27)
+				)
+			)
+		)
+		(property "Datasheet" ""
+			(at 171.45 63.5 0)
+			(hide yes)
+			(show_name no)
+			(do_not_autoplace no)
+			(effects
+				(font
+					(size 1.27 1.27)
+				)
+			)
+		)
+		(property "Description" "Power symbol creates a global label with name \"GND\" , ground"
+			(at 171.45 63.5 0)
+			(hide yes)
+			(show_name no)
+			(do_not_autoplace no)
+			(effects
+				(font
+					(size 1.27 1.27)
+				)
+			)
+		)
+		(pin "1"
+		)
+		(instances
+			(project "Carry"
+				(path "/460b64f1-754e-43cc-bbda-1ad83299f772"
+					(reference "#PWR07")
+					(unit 1)
+				)
+			)
+		)
+	)
+	(symbol
+		(lib_id "power:GND")
 		(at 92.71 50.8 270)
 		(unit 1)
@@
 					(unit 1)
 				)
+			)
+		)
+	)
+	(symbol
+		(lib_id "power:GND")
+		(at 140.97 63.5 270)
+		(unit 1)
+		(body_style 1)
+		(exclude_from_sim no)
+		(in_bom yes)
+		(on_board yes)
+		(in_pos_files yes)
+		(dnp no)
+		(fields_autoplaced yes)
+		(property "Reference" "#PWR05"
+			(at 134.62 63.5 0)
+			(hide yes)
+			(show_name no)
+			(do_not_autoplace no)
+			(effects
+				(font
+					(size 1.27 1.27)
+				)
+			)
+		)
+		(property "Value" "GND"
+			(at 137.16 63.4999 90)
+			(show_name no)
+			(do_not_autoplace no)
+			(effects
+				(font
+					(size 1.27 1.27)
+				)
+				(justify right)
+			)
+		)
+		(property "Footprint" ""
+			(at 140.97 63.5 0)
+			(hide yes)
+			(show_name no)
+			(do_not_autoplace no)
+			(effects
+				(font
+					(size 1.27 1.27)
+				)
+			)
+		)
+		(property "Datasheet" ""
+			(at 140.97 63.5 0)
+			(hide yes)
+			(show_name no)
+			(do_not_autoplace no)
+			(effects
+				(font
+					(size 1.27 1.27)
+				)
+			)
+		)
+		(property "Description" "Power symbol creates a global label with name \"GND\" , ground"
+			(at 140.97 63.5 0)
+			(hide yes)
+			(show_name no)
+			(do_not_autoplace no)
+			(effects
+				(font
+					(size 1.27 1.27)
+				)
+			)
+		)
+		(pin "1"
+		)
+		(instances
+			(project "Carry"
+				(path "/460b64f1-754e-43cc-bbda-1ad83299f772"
+					(reference "#PWR05")
+					(unit 1)
+				)

Commit message: updated
Parts:
- removed D1: LED, symbol Device:LED
- added C1, C2: 4.7, symbol Device:C
- added D1: LED_Dual_AAK, LED_SMD:LED-L1T2_LUMILEDS, symbol Device:LED_Dual_AAK
- added J1: Conn_01x04_Pin, symbol Connector:Conn_01x04_Pin
- added R3: 330, symbol Device:R
- added R4: 1k, symbol Device:R
- R2: value 1k -> 470
Connections:
- net GND: now also C1.2, C2.2, D1.3 (K), J1.4 (Pin_4)
- net at J2.1 (Pin_1), U1.1 (VBUS), U2.3 (V_{BAT})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: now also R2.2, C1.1, C2.1, J1.1 (Pin_1)
- net at U1.20 (GPIO4_C1_z): now also R3.2
- net at R2.1: now also U2.1 (STAT), R4.1
- new net: D1.1 (A1), R4.2
- new net: D1.2 (A2), R3.1
- new net D+: J1.3 (Pin_3)
- new net D-: J1.2 (Pin_2)
- no-connect marks 15 -> 16
